Commit message: [robotiq_2f_140_gripper_visualization] Added Gazebo materials and mimic joint plugin
Ideally we'd implement an articlated_gazebo_plugin as for the 3f
gripper. For now it's adding the materials and a mimic joint plugin
using
https://github.com/roboticsgroup/roboticsgroup_upatras_gazebo_plugins.git

File: robotiq_2f_140_gripper_visualization/urdf/robotiq_arg2f_140_model_macro.xacro (robot description, xacro)
@@ -2,4 +2,5 @@
 <robot xmlns:xacro="http://ros.org/wiki/xacro">
   <xacro:include filename="$(find robotiq_2f_140_gripper_visualization)/urdf/robotiq_arg2f_transmission.xacro" />
+  <xacro:include filename="$(find robotiq_2f_140_gripper_visualization)/urdf/robotiq_arg2f_gazebo.xacro" />
   <xacro:macro name="outer_knuckle" params="prefix fingerprefix stroke">
     <link name="${prefix}${fingerprefix}_outer_knuckle">
@@ -203,5 +204,5 @@
     <xacro:finger_joints prefix="${prefix}" fingerprefix="right" reflect="-1.0"/>
   </xacro:macro>
-  <xacro:macro name="robotiq_arg2f_140" params="prefix">
+  <xacro:macro name="robotiq_arg2f_140" params="prefix gazebo:=true">
     <xacro:robotiq_arg2f_base_link prefix="${prefix}"/>
     <xacro:finger_links prefix="${prefix}" fingerprefix="left" stroke="140"/>
@@ -210,4 +211,7 @@
     <xacro:right_outer_knuckle_joint prefix="${prefix}"/>
     <xacro:robotiq_arg2f_transmission prefix="${prefix}"/>
+    <xacro:if value="${gazebo}">
+      <xacro:robotiq_arg2f_gazebo prefix="${prefix}"/>
+    </xacro:if>
   </xacro:macro>
 </robot>

Commit message: [robotiq_2f_gripper_visualization] Remove unsupported collision/material tag

File: robotiq_2f_140_gripper_visualization/urdf/robotiq_arg2f_140_model_macro.xacro (robot description, xacro)
@@ -140,7 +140,4 @@
            <box size="0.03 0.07 0.0075"/>
         </geometry>
-        <material name="">
-          <color rgba="0.9 0.0 0.0 1" />
-        </material>
       </collision>
     </link>
