Commit message: [robotiq_ft_sensor] Add primitive shape collision model (cylinders)

File: robotiq_ft_sensor/urdf/robotiq_ft300.urdf.xacro (robot description, xacro)
@@ -37,7 +37,9 @@
             </visual>
             <collision>
-                <origin xyz="0 0 0" rpy="0 0 0" />
+                <!-- <origin xyz="0 0 0" rpy="0 0 0" /> -->
+                <origin xyz="0 0 ${0.035/2}" rpy="0 0 0" />
                 <geometry>
-                    <mesh filename="package://robotiq_ft_sensor/meshes/collision/robotiq_ft300.STL"/>
+                    <cylinder length="0.035" radius="${0.075/2}"/>
+                    <!-- <mesh filename="package://robotiq_ft_sensor/meshes/collision/robotiq_ft300.STL"/> -->
                 </geometry>
             </collision>
@@ -55,7 +57,9 @@
             </visual>
             <collision>
-                <origin xyz="0 0 0" rpy="0 0 0" />
+                <!-- <origin xyz="0 0 0" rpy="0 0 0" /> -->
+                <origin xyz="0 0 ${0.013/2}" rpy="0 0 0" />
                 <geometry>
-                    <mesh filename="package://robotiq_ft_sensor/meshes/collision/mountings/robotiq_ft300-G-062-COUPLING_G-50-4M6-1D6_20181119.STL"/>
+                    <cylinder length="0.013" radius="${0.075/2}"/>
+                    <!-- <mesh filename="package://robotiq_ft_sensor/meshes/collision/mountings/robotiq_ft300-G-062-COUPLING_G-50-4M6-1D6_20181119.STL"/> -->
                 </geometry>
             </collision>

Commit message: [robotiq_ft_sensor] Fix typo

File: robotiq_ft_sensor/urdf/robotiq_ft300.urdf.xacro (robot description, xacro)
@@ -77,5 +77,5 @@
                 points the opposite way away from the connector.
             - The Y axis uses the right hand thumb rule according to X-Z. -->
-        <joint name="${prefix}measurment_joint" type="fixed">
+        <joint name="${prefix}measurement_joint" type="fixed">
             <origin xyz="0 0 0" rpy="0 ${pi} ${-pi/2}" />
             <parent link="${prefix}ft300_sensor" />

File: robotiq_ft_sensor/urdf/robotiq_fts150.urdf.xacro (robot description, xacro)
@@ -30,5 +30,5 @@
         </link>
         <!-- virtual measurement frame -->
-        <joint name="${prefix}measurment_joint" type="fixed" >
+        <joint name="${prefix}measurement_joint" type="fixed" >
             <origin xyz="0 0 0.01625" rpy="0 0 0" />
             <parent link="${prefix}fts_robotside" />

Commit message: Rename joint to avoid joint and link name clash (Pinocchio bug)

File: robotiq_ft_sensor/urdf/robotiq_ft300.urdf.xacro (robot description, xacro)
@@ -66,5 +66,5 @@
         </link>
          <!-- Connect force sensor with mounting/coupling plate -->
-        <joint name="${prefix}ft300_mounting_plate" type="fixed">
+        <joint name="${prefix}ft300_mounting_plate_joint" type="fixed">
             <origin xyz="0 0 0.0415" rpy="0 ${pi} 0"/>
             <parent link="${prefix}ft300_mounting_plate" />

Commit message: [robotiq_ft_sensor] Add Gazebo materials to FT300

File: robotiq_ft_sensor/urdf/robotiq_ft300.urdf.xacro (robot description, xacro)
@@ -45,4 +45,7 @@
             </collision>
         </link>
+        <gazebo reference="${prefix}ft300_sensor">
+            <material>Gazebo/Black</material>
+        </gazebo>
         <!-- Link representing the FT300 mounting plate -->
         <link name="${prefix}ft300_mounting_plate">
@@ -65,4 +68,7 @@
             </collision>
         </link>
+        <gazebo reference="${prefix}ft300_mounting_plate">
+            <material>Gazebo/Black</material>
+        </gazebo>
          <!-- Connect force sensor with mounting/coupling plate -->
         <joint name="${prefix}ft300_mounting_plate_joint" type="fixed">

Commit message: [robotiq_ft_sensor] Remove unsupported tags in inertial

File: robotiq_ft_sensor/urdf/robotiq_ft300.urdf.xacro (robot description, xacro)
@@ -25,5 +25,5 @@
                 <origin xyz="0 0 ${-17 / 1000}" rpy="0 0 0"/>
                 <mass value="0.300"/>
-                <inertia ixx="${262 / 1000000}" ixy="0" ixz="${1 / 1000000}" iyy="${265 / 1000000}" iyx="0" iyz="${1 / 1000000}" izz="${219 / 1000000}" izx="${-1 / 1000000}" izy="${1 / 1000000}"/>
+                <inertia ixx="${262 / 1000000}" ixy="0" ixz="${1 / 1000000}" iyy="${265 / 1000000}" iyz="${1 / 1000000}" izz="${219 / 1000000}"/>
             </inertial>
             <visual>

Commit message: [robotiq_ft_sensor] Add Gazebo F/T plug-in
This required changing the joint type from fixed to revolute/prismatic
with zero limits

File: robotiq_ft_sensor/urdf/robotiq_ft300.urdf.xacro (robot description, xacro)
@@ -83,10 +83,35 @@
                 points the opposite way away from the connector.
             - The Y axis uses the right hand thumb rule according to X-Z. -->
-        <joint name="${prefix}measurement_joint" type="fixed">
+        <!-- Defined as a revolute joint with no motion to enable force/torque sensing -->
+        <joint name="${prefix}measurement_joint" type="revolute">
             <origin xyz="0 0 0" rpy="0 ${pi} ${-pi/2}" />
             <parent link="${prefix}ft300_sensor" />
             <child link="${prefix}robotiq_ft_frame_id" />
+            <limit velocity="100.0" effort="300.0" lower="0" upper="0" />
         </joint>
         <link name="${prefix}robotiq_ft_frame_id"/>
+        <!-- Gazebo: Simulation of force-torque sensor -->
+        <gazebo reference="${prefix}measurement_joint">
+            <provideFeedback>true</provideFeedback>
+            <gravity>true</gravity>
+        </gazebo>
+        <gazebo>
+            <plugin name="ft_sensor" filename="libgazebo_ros_ft_sensor.so">
+                <updateRate>100.0</updateRate>
+                <topicName>${prefix}robotiq_ft_wrench</topicName>
+                <jointName>${prefix}measurement_joint</jointName>
+                <gaussianNoise>0.003</gaussianNoise>
+            </plugin>
+        </gazebo>
+        <transmission name="${prefix}measurement_joint_trans">
+            <type>transmission_interface/SimpleTransmission</type>
+            <joint name="${prefix}measurement_joint">
+            <!-- <hardwareInterface>hardware_interface/ForceTorqueSensorInterface</hardwareInterface> -->
+            <hardwareInterface>hardware_interface/PositionJointInterface</hardwareInterface>
+            </joint>
+            <actuator name="${prefix}measurement_joint_motor">
+                <mechanicalReduction>1</mechanicalReduction>
+            </actuator>
+        </transmission>
     </xacro:macro>
 </robot>

Commit message: [robotiq_ft_sensor] Add gazebo flag to macro to turn off Gazebo-specific modifications
The revolute joint for simulating the force/torque is a Gazebo-specific
hack and should not be used on hardware

File: robotiq_ft_sensor/urdf/robotiq_ft300.urdf.xacro (robot description, xacro)
@@ -13,5 +13,5 @@
         ```
     -->
-    <xacro:macro name="robotiq_ft300" params="parent prefix *origin">
+    <xacro:macro name="robotiq_ft300" params="parent prefix *origin gazebo:=false">
         <!-- mount the fts to the robot -->
         <joint name="${prefix}ft300_fix" type="fixed">
@@ -45,7 +45,4 @@
             </collision>
         </link>
-        <gazebo reference="${prefix}ft300_sensor">
-            <material>Gazebo/Black</material>
-        </gazebo>
         <!-- Link representing the FT300 mounting plate -->
         <link name="${prefix}ft300_mounting_plate">
@@ -68,7 +65,4 @@
             </collision>
         </link>
-        <gazebo reference="${prefix}ft300_mounting_plate">
-            <material>Gazebo/Black</material>
-        </gazebo>
          <!-- Connect force sensor with mounting/coupling plate -->
         <joint name="${prefix}ft300_mounting_plate_joint" type="fixed">
@@ -83,35 +77,54 @@
                 points the opposite way away from the connector.
             - The Y axis uses the right hand thumb rule according to X-Z. -->
-        <!-- Defined as a revolute joint with no motion to enable force/torque sensing -->
-        <joint name="${prefix}measurement_joint" type="revolute">
-            <origin xyz="0 0 0" rpy="0 ${pi} ${-pi/2}" />
-            <parent link="${prefix}ft300_sensor" />
-            <child link="${prefix}robotiq_ft_frame_id" />
-            <limit velocity="100.0" effort="300.0" lower="0" upper="0" />
-        </joint>
+        <!-- Hardware: Fixed joint -->
+        <xacro:unless value="${gazebo}">
+            <joint name="${prefix}measurement_joint" type="fixed">
+                <origin xyz="0 0 0" rpy="0 ${pi} ${-pi/2}" />
+                <parent link="${prefix}ft300_sensor" />
+                <child link="${prefix}robotiq_ft_frame_id" />
+            </joint>
+        </xacro:unless>
+        <!-- Gazebo: Defined as a revolute joint with no motion to enable force/torque sensing -->
+        <xacro:if value="${gazebo}">
+            <joint name="${prefix}measurement_joint" type="revolute">
+                <origin xyz="0 0 0" rpy="0 ${pi} ${-pi/2}" />
+                <parent link="${prefix}ft300_sensor" />
+                <child link="${prefix}robotiq_ft_frame_id" />
+                <limit velocity="100.0" effort="300.0" lower="0" upper="0" />
+            </joint>
+        </xacro:if>
         <link name="${prefix}robotiq_ft_frame_id"/>
-        <!-- Gazebo: Simulation of force-torque sensor -->
-        <gazebo reference="${prefix}measurement_joint">
-            <provideFeedback>true</provideFeedback>
-            <gravity>true</gravity>
-        </gazebo>
-        <gazebo>
-            <plugin name="ft_sensor" filename="libgazebo_ros_ft_sensor.so">
-                <updateRate>100.0</updateRate>
-                <topicName>${prefix}robotiq_ft_wrench</topicName>
-                <jointName>${prefix}measurement_joint</jointName>
-                <gaussianNoise>0.003</gaussianNoise>
-            </plugin>
-        </gazebo>
-        <transmission name="${prefix}measurement_joint_trans">
-            <type>transmission_interface/SimpleTransmission</type>
-            <joint name="${prefix}measurement_joint">
-            <!-- <hardwareInterface>hardware_interface/ForceTorqueSensorInterface</hardwareInterface> -->
-            <hardwareInterface>hardware_interface/PositionJointInterface</hardwareInterface>
-            </joint>
-            <actuator name="${prefix}measurement_joint_motor">
-                <mechanicalReduction>1</mechanicalReduction>
-            </actuator>
-        </transmission>
+        <!-- Gazebo settings -->
+        <xacro:if value="${gazebo}">
+            <gazebo reference="${prefix}ft300_sensor">
+                <material>Gazebo/Black</material>
+            </gazebo>
+            <gazebo reference="${prefix}ft300_mounting_plate">
+                <material>Gazebo/Black</material>
+            </gazebo>
+            <!-- Gazebo: Simulation of force-torque sensor -->
+            <gazebo reference="${prefix}measurement_joint">
+                <provideFeedback>true</provideFeedback>
+                <gravity>true</gravity>
+            </gazebo>
+            <gazebo>
+                <plugin name="ft_sensor" filename="libgazebo_ros_ft_sensor.so">
+                    <updateRate>100.0</updateRate>
+                    <topicName>${prefix}robotiq_ft_wrench</topicName>
+                    <jointName>${prefix}measurement_joint</jointName>
+                    <gaussianNoise>0.003</gaussianNoise>
+                </plugin>
+            </gazebo>
+            <transmission name="${prefix}measurement_joint_trans">
+                <type>transmission_interface/SimpleTransmission</type>
+                <joint name="${prefix}measurement_joint">
+                <!-- <hardwareInterface>hardware_interface/ForceTorqueSensorInterface</hardwareInterface> -->
+                <hardwareInterface>hardware_interface/PositionJointInterface</hardwareInterface>
+                </joint>
+                <actuator name="${prefix}measurement_joint_motor">
+                    <mechanicalReduction>1</mechanicalReduction>
+                </actuator>
+            </transmission>
+        </xacro:if>
     </xacro:macro>
 </robot>

Commit message: [robotiq_ft_sensor] Add option to specify topicName for FT sensor

File: robotiq_ft_sensor/urdf/robotiq_ft300.urdf.xacro (robot description, xacro)
@@ -1,5 +1,5 @@
 <?xml version="1.0"?>
 <!-- Developed by: Daniel Ordonez 20.06.2019 - daniels.ordonez@gmail.com-->
-<robot xmlns:xacro="http://ros.org/wiki/xacro" name="robotiq_fts150">
+<robot xmlns:xacro="http://ros.org/wiki/xacro" name="robotiq_ft300">
     <!-- Macro function to instanciate URDF model of the FT300 force-torque sensor with mounting plate
         Example use:
@@ -13,5 +13,5 @@
         ```
     -->
-    <xacro:macro name="robotiq_ft300" params="parent prefix *origin gazebo:=false">
+    <xacro:macro name="robotiq_ft300" params="parent prefix *origin gazebo:=false ft_topic:=''">
         <!-- mount the fts to the robot -->
         <joint name="${prefix}ft300_fix" type="fixed">
@@ -111,5 +111,10 @@
                 <plugin name="ft_sensor" filename="libgazebo_ros_ft_sensor.so">
                     <updateRate>100.0</updateRate>
+                    <xacro:if value="${ft_topic!=''}">
+                    <topicName>${ft_topic}</topicName>
+                    </xacro:if>
+                    <xacro:if value="${ft_topic==''}">
                     <topicName>${prefix}robotiq_ft_wrench</topicName>
+                    </xacro:if>
                     <jointName>${prefix}measurement_joint</jointName>
                     <gaussianNoise>0.003</gaussianNoise>
